Commit message: perf(A1-ROS2):Mercury A1 updated URDF model file

File: mercury_description/urdf/mercury_a1/mercury_a1_old.urdf (robot description, URDF)
Before this commit: robot firefighter, 8 links, 7 joints
Links:
- link base: geometry collision cylinder length=0.07 radius=0.043; visual mesh filename=package://mercury_description/urdf/mercury_a1/base.dae
- link joint1: geometry collision cylinder length=0.02 radius=0.023; visual mesh filename=package://mercury_description/urdf/mercury_a1/joint1.dae
- link joint2: geometry collision cylinder length=0.035 radius=0.023; visual mesh filename=package://mercury_description/urdf/mercury_a1/joint2.dae
- link joint3: geometry collision cylinder length=0.02 radius=0.023; visual mesh filename=package://mercury_description/urdf/mercury_a1/joint3.dae
- link joint4: geometry collision cylinder length=0.035 radius=0.023; visual mesh filename=package://mercury_description/urdf/mercury_a1/joint4.dae
- link joint5: geometry collision cylinder length=0.06 radius=0.023; visual mesh filename=package://mercury_description/urdf/mercury_a1/joint5.dae
Joints:
- joint joint1_to_base: origin xyz=0 0 0.17835 rpy=0 0 0 -> xyz=0 0 0.175 rpy=0 0 0
- joint joint2_to_joint1: limit lower=-0.8726 upper=2.0943 effort=1000.0 velocity=0 -> lower=-0.959 upper=1.658 effort=1000.0 velocity=0; origin xyz=0 -0.005 -0.01 rpy=-1.5708 0 0 -> xyz=0 0  0 rpy=-1.5708 0 0
- joint joint3_to_joint2: origin xyz=0 -0.134 0.004    rpy=1.5708 0 0 -> xyz=0 -0.11 0    rpy=1.5708 0 0
- joint joint4_to_joint3: limit lower=-2.879 upper=0.087 effort=1000.0 velocity=0 -> lower=-3.019 upper=0.087 effort=1000.0 velocity=0; origin xyz=0.03 0 0.07 rpy=-1.5708 0 3.14159 -> xyz=0.03 0 0.095 rpy=-1.5708 0 3.14159
- joint joint5_to_joint4: origin xyz=0.031 -0.11 0 rpy=1.5708 3.14159 0 -> xyz=0.03 -0.126 0 rpy=1.5708 3.14159 0
- joint joint6_to_joint5: limit lower=-0.3490 upper=4.6251 effort=1000.0 velocity=0 -> lower=-0.0349 upper=2.9321 effort=1000.0 velocity=0; origin xyz=0 0.03 0.095 rpy=1.5708 0 0 -> xyz=0 0.0 0.08 rpy=1.5708 0 0
- joint joint7_to_joint6: origin xyz=0.038 -0.045 0.025 rpy=1.5708 0 0 -> xyz=0.038 -0.046 0 rpy=1.5708 0 0
