Commit message: Update mercury_b1.urdf joint limit rang

File: mercury_description/urdf/mercury_b1/mercury_b1.urdf (robot description, URDF)
Before this commit: robot firefighter, 18 links, 17 joints
Joints:
- joint joint2_L: limit lower=-0.959 upper=1.658 effort=1000.0 velocity=0 -> lower=-0.8726 upper=2.0943 effort=1000.0 velocity=0
- joint joint2_R: limit lower=-0.959 upper=1.658 effort=1000.0 velocity=0 -> lower=-0.8726 upper=2.0943 effort=1000.0 velocity=0
- joint joint4_L: limit lower=-3.019 upper=0.087 effort=1000.0 velocity=0 -> lower=-2.879 upper=0.087 effort=1000.0 velocity=0
- joint joint4_R: limit lower=-3.019 upper=0.087 effort=1000.0 velocity=0 -> lower=-2.879 upper=0.087 effort=1000.0 velocity=0
