Commit message: feat(E1-URDF):E1 Added ROS2 URDF-controllable model.

File: mercury_description/urdf/mercury_e1/mercury_e1.urdf (robot description, URDF)
Before this commit: robot MercuyrE1, 1 links, 0 joints
Links:
- removed link base
- added link J1_Link, mass 1.01999225695505; collision mesh filename=package://mercury_description/urdf/mercury_e1/J1_Link.STL; visual mesh filename=package://mercury_description/urdf/mercury_e1/J1_Link.STL
- added link J2_Link, mass 0.865977615667264; collision mesh filename=package://mercury_description/urdf/mercury_e1/J2_Link.STL; visual mesh filename=package://mercury_description/urdf/mercury_e1/J2_Link.STL
- added link J3_Link, mass 0.562852488998004; collision mesh filename=package://mercury_description/urdf/mercury_e1/J3_Link.STL; visual mesh filename=package://mercury_description/urdf/mercury_e1/J3_Link.STL
- added link J4_Link, mass 0.688296580358887; collision mesh filename=package://mercury_description/urdf/mercury_e1/J4_Link.STL; visual mesh filename=package://mercury_description/urdf/mercury_e1/J4_Link.STL
- added link J5_Link, mass 0.410203464751654; collision mesh filename=package://mercury_description/urdf/mercury_e1/J5_Link.STL; visual mesh filename=package://mercury_description/urdf/mercury_e1/J5_Link.STL
- added link J6_Link, mass 0.98; collision mesh filename=package://mercury_description/urdf/mercury_e1/J6_Link.STL; visual mesh filename=package://mercury_description/urdf/mercury_e1/J6_Link.STL
- added link J7_Link, mass 0.158638180498606; collision mesh filename=package://mercury_description/urdf/mercury_e1/J7_Link.STL; visual mesh filename=package://mercury_description/urdf/mercury_e1/J7_Link.STL
- added link base_link, mass 1.31191278229374; collision mesh filename=package://mercury_description/urdf/mercury_e1/base_link.STL; visual mesh filename=package://mercury_description/urdf/mercury_e1/base_link.STL
Joints:
- added joint J1: type revolute, parent base_link, child J1_Link, origin xyz=-0.000749999816993875 0.0374529801453609 -0.465449956874081 rpy=0 0 0, axis 0 0 -1, limit lower=-2.7 upper=2.7 effort=0 velocity=0
- added joint J2: type revolute, parent J1_Link, child J2_Link, origin xyz=0 -0.0365011426633475 -0.0292499753403238 rpy=0 0 0, axis 0 1 0, limit lower=-0.96 upper=1.83 effort=0 velocity=0
- added joint J3: type revolute, parent J2_Link, child J3_Link, origin xyz=0.000749999999985258 0.0365481432413965 0.156250000000001 rpy=0 0 0, axis 0 0 -1, limit lower=-2.79 upper=2.79 effort=0 velocity=0
- added joint J4: type revolute, parent J3_Link, child J4_Link, origin xyz=0.0149999999999998 -0.0389999807242169 0.111 rpy=0 0 0, axis 0 1 0, limit lower=-0.314 upper=2.356 effort=0 velocity=0
- added joint J5: type revolute, parent J4_Link, child J5_Link, origin xyz=-0.0149999999999995 0.0390000000000039 0.11995 rpy=0 0 0, axis 0 0 -1, limit lower=-2.79 upper=2.79 effort=0 velocity=0
- added joint J6: type revolute, parent J5_Link, child J6_Link, origin xyz=0 -0.0374999999991969 0.107499932214404 rpy=0 0 0, axis 0 -1 0, limit lower=-2.042 upper=1.745 effort=0 velocity=0
- added joint J7: type revolute, parent J6_Link, child J7_Link, origin xyz=0 0.037499986816365 0.0819499999999993 rpy=0 0 0, axis 0 0 1, limit lower=-2.356 upper=2.356 effort=0 velocity=0

Commit message: perf(E1-URDF): opt E1 urdf file

File: mercury_description/urdf/mercury_e1/mercury_e1.urdf (robot description, URDF)
Before this commit: robot MercuryE1, 8 links, 7 joints
Links:
- added link dummy_link
Joints:
- removed joint J1
- removed joint J2
- removed joint J3
- removed joint J4
- removed joint J5
- removed joint J6
- removed joint J7
- added joint Joint1: type revolute, parent base_link, child J1_Link, origin xyz=0 0 0.255 rpy=0 0 0, axis 0 0 -1, limit lower=-2.7 upper=2.7 effort=10000 velocity=2
- added joint Joint2: type revolute, parent J1_Link, child J2_Link, origin xyz=0 -0.0365011426633475 -0.0292499753403238 rpy=0 0 0, axis 0 1 0, limit lower=-0.96 upper=1.83 effort=10000 velocity=2
- added joint Joint3: type revolute, parent J2_Link, child J3_Link, origin xyz=0.000749999999985258 0.0365481432413965 0.156250000000001 rpy=0 0 0, axis 0 0 -1, limit lower=-2.79 upper=2.79 effort=10000 velocity=2
- added joint Joint4: type revolute, parent J3_Link, child J4_Link, origin xyz=0.0149999999999998 -0.0389999807242169 0.111 rpy=0 0 0, axis 0 -1 0, limit lower=-2.35 upper=0.314 effort=10000 velocity=2
- added joint Joint5: type revolute, parent J4_Link, child J5_Link, origin xyz=-0.0149999999999995 0.0390000000000039 0.11995 rpy=0 0 0, axis 0 0 -1, limit lower=-2.79 upper=2.79 effort=10000 velocity=2
- added joint Joint6: type revolute, parent J5_Link, child J6_Link, origin xyz=0 -0.0374999999991969 0.107499932214404 rpy=0 0 0, axis 0 -1 0, limit lower=-1.74 upper=2.042 effort=10000 velocity=2
- added joint Joint7: type revolute, parent J6_Link, child J7_Link, origin xyz=0 0.037499986816365 0.0819499999999993 rpy=0 0 0, axis 0 0 1, limit lower=-2.35 upper=2.35 effort=10000 velocity=2
- added joint dummy: type fixed, parent dummy_link, child base_link

Commit message: perf(E1-URDF):Update the rotation direction of the urdf joint

File: mercury_description/urdf/mercury_e1/mercury_e1.urdf (robot description, URDF)
Before this commit: robot MercuryE1, 9 links, 8 joints
Joints:
- joint Joint1: axis 0 0 -1 -> 0 0 1
- joint Joint3: axis 0 0 -1 -> 0 0 1
- joint Joint5: axis 0 0 -1 -> 0 0 1
